Commit message: add onArm_camera

File: Pickbot_with_moveit/universal_robot/ur_description/urdf/ur.gazebo.xacro (robot description, xacro)
@@ -23,4 +23,47 @@
       <selfCollide>true</selfCollide>
     </gazebo>
+    <!-- INTEL REALSENSE DEPTH CAMERA -->
+    <gazebo reference="${prefix}camera_link2">
+      <sensor name="camera" type="depth">
+        <always_on>true</always_on>
+        <update_rate>20.0</update_rate>
+        <camera>
+          <horizontal_fov>1.57</horizontal_fov>
+          <image>
+            <format>R8G8B8</format>
+            <width>640</width>
+            <height>480</height>
+          </image>
+          <clip>
+            <near>0.01</near>
+            <far>8.0</far>
+          </clip>
+        </camera>
+        <plugin filename="libgazebo_ros_openni_kinect.so" name="depth_camera">
+          <cameraName>intel_realsense_camera</cameraName>
+          <alwaysOn>true</alwaysOn>
+          <updateRate>10</updateRate>
+          <imageTopicName>rgb/image_raw</imageTopicName>
+          <depthImageTopicName>depth/image_raw</depthImageTopicName>
+          <pointCloudTopicName>depth/points</pointCloudTopicName>
+          <cameraInfoTopicName>rgb/camera_info</cameraInfoTopicName>
+          <depthImageCameraInfoTopicName>depth/camera_info</depthImageCameraInfoTopicName>
+          <frameName>camera_depth_optical_frame</frameName>
+          <baseline>0.1</baseline>
+          <distortion_k1>0.0</distortion_k1>
+          <distortion_k2>0.0</distortion_k2>
+          <distortion_k3>0.0</distortion_k3>
+          <distortion_t1>0.0</distortion_t1>
+          <distortion_t2>0.0</distortion_t2>
+          <pointCloudCutoff>0.4</pointCloudCutoff>
+          <!--pointCloudCutoffMax>2</pointCloudCutoffMax-->
+          <!--CxPrime>0</CxPrime-->
+          <!--Cx>0</Cx-->
+          <!--Cy>0</Cy-->
+          <!--focalLength>320.254926</focalLength-->
+          <!--hackBaseline>0</hackBaseline-->
+        </plugin>
+      </sensor>
+    </gazebo>
   </xacro:macro>
 </robot>

File: Pickbot_with_moveit/universal_robot/ur_description/urdf/ur10.urdf.xacro (robot description, xacro)
@@ -316,4 +316,50 @@
       <child link="${prefix}tool0"/>
     </joint>
+    <!-- INTEL REALSENSE DEPTH CAMERA -->
+    <joint name="${prefix}camera_rgb_joint" type="fixed">
+      <!-- <origin rpy="0 0.785 3.14" xyz="1 1 0.75"/> fixed camera -->
+      <!-- <parent link="base_link"/> fixed camera -->
+      <!-- <origin rpy="0 -1.57 -1.57" xyz="0 0.21 0.078"/> -->
+      <origin rpy="0 -0.9 1.57" xyz="0 0.21 -0.078"/>
+      <parent link="${prefix}wrist_3_link"/>
+      <child link="${prefix}camera_rgb_frame"/>
+    </joint>
+    <link name="${prefix}camera_rgb_frame"/>
+    <joint name="${prefix}camera_rgb_optical_joint" type="fixed">
+      <origin rpy="-1.57079632679 0 -1.57079632679" xyz="0 0 0"/>
+      <parent link="${prefix}camera_rgb_frame"/>
+      <child link="${prefix}camera_rgb_optical_frame"/>
+    </joint>
+    <link name="${prefix}camera_rgb_optical_frame"/>
+    <joint name="${prefix}camera_joint2" type="fixed">
+      <origin rpy="0 0 0" xyz="0 0 0"/>
+      <parent link="${prefix}camera_rgb_frame"/>
+      <child link="${prefix}camera_link2"/>
+    </joint>
+    <link name="${prefix}camera_link2">
+      <visual>
+        <origin rpy="0 0 1.57079632679" xyz="0 0 0"/>
+        <geometry>
+          <mesh filename="package://ur_description/meshes/intel_realsense/intel_realsense_camera.DAE"/>
+        </geometry>
+      </visual>
+      <!-- <inertial>
+        <mass value="0.564"/>
+        <origin xyz="0 0 0"/>
+        <inertia ixx="0.003881243" ixy="0.0" ixz="0.0" iyy="0.000498940" iyz="0.0" izz="0.003879257"/>
+      </inertial> -->
+    </link>
+    <joint name="${prefix}camera_depth_joint" type="fixed">
+      <origin rpy="0 0 0" xyz="0 0 0"/>
+      <parent link="${prefix}camera_rgb_frame"/>
+      <child link="${prefix}camera_depth_frame"/>
+    </joint>
+    <link name="${prefix}camera_depth_frame"/>
+    <joint name="${prefix}camera_depth_optical_joint" type="fixed">
+      <origin rpy="-1.57079632679 0 -1.57079632679" xyz="0 0 0"/>
+      <parent link="${prefix}camera_depth_frame"/>
+      <child link="${prefix}camera_depth_optical_frame"/>
+    </joint>
+    <link name="${prefix}camera_depth_optical_frame"/>
   </xacro:macro>
 </robot>

Commit message: add 2 collision sensors

File: Pickbot_with_moveit/universal_robot/ur_description/urdf/ur.gazebo.xacro (robot description, xacro)
@@ -22,4 +22,46 @@
     <gazebo reference="${prefix}ee_link">
       <selfCollide>true</selfCollide>
+    </gazebo>
+    <!-- COLLISION/BUMPER SENSOR 1 LINK JOINT PLUGIN-->
+    <gazebo reference="${prefix}gripper_contactsensor_link_1">
+      <kp>1000.0</kp>
+      <kd>1000.0</kd>
+      <mu1>100000000000000000.0</mu1>
+      <mu2>100000000000000000.0</mu2>
+      <material>Gazebo/Red</material>
+    </gazebo>
+    <gazebo reference="${prefix}gripper_contactsensor_link_1">
+      <sensor name="gripper_contactsensor_sensor_1" type="contact">
+        <always_on>true</always_on>
+        <!--<update_rate>30</update_rate>-->
+        <contact>
+          <collision>wrist_3_link_fixed_joint_lump__gripper_contactsensor_link_1_collision_2</collision>
+        </contact>
+        <plugin name="bumper0_plugin" filename="libgazebo_ros_bumper.so">
+          <bumperTopicName>gripper_contactsensor_1_state</bumperTopicName>
+          <frameName>gripper_contactsensor_link_1</frameName>
+        </plugin>
+      </sensor>
+    </gazebo>
+    <!-- COLLISION/BUMPER SENSOR 2 LINK JOINT PLUGIN-->
+    <gazebo reference="${prefix}gripper_contactsensor_link_2">
+      <kp>1000.0</kp>
+      <kd>1000.0</kd>
+      <mu1>100000000000000000.0</mu1>
+      <mu2>100000000000000000.0</mu2>
+      <material>Gazebo/Red</material>
+    </gazebo>
+    <gazebo reference="${prefix}gripper_contactsensor_link_2">
+      <sensor name="gripper_contactsensor_sensor_2" type="contact">
+        <always_on>true</always_on>
+        <!--<update_rate>30</update_rate>-->
+        <contact>
+          <collision>wrist_3_link_fixed_joint_lump__gripper_contactsensor_link_2_collision_3</collision>
+        </contact>
+        <plugin name="bumper0_plugin" filename="libgazebo_ros_bumper.so">
+          <bumperTopicName>gripper_contactsensor_2_state</bumperTopicName>
+          <frameName>gripper_contactsensor_link_2</frameName>
+        </plugin>
+      </sensor>
     </gazebo>
     <!-- INTEL REALSENSE DEPTH CAMERA -->

File: Pickbot_with_moveit/universal_robot/ur_description/urdf/ur10.urdf.xacro (robot description, xacro)
@@ -316,4 +316,60 @@
       <child link="${prefix}tool0"/>
     </joint>
+<!-- COLLISION/BUMPER SENSOR 1 LINK JOINT PLUGIN-->
+    <link name="${prefix}gripper_contactsensor_link_1">
+      <inertial >
+            <origin xyz="0 0 0" rpy="0 0 0"/>
+            <mass value="0.0001" />
+            <inertia ixx="1.6e-08" ixy="0.0" ixz="0.0" iyy="1.6e-08" iyz="0.0" izz="1.6e-08"/>
+        </inertial>
+        <collision>
+            <origin xyz="0 0 0" rpy="0 0 0"/>
+            <geometry>
+                <box size="0.02 0.02 0.0001"/>
+            </geometry>
+        </collision>
+        <visual>
+            <origin rpy="0.0 0 0" xyz="0 0 0"/>
+            <geometry>
+                <box size="0.02 0.02 0.0001"/>
+            </geometry>
+            <material name="red">
+              <color rgba="1.0 0 0 1.0"/>
+          </material>
+        </visual>
+    </link>
+    <joint name="${prefix}gripper_contactsensor_link_1_joint" type="fixed">
+      <origin xyz="-0.019 0.296 0.0" rpy="1.570796325 0 0"/>
+      <parent link="${prefix}wrist_3_link"/>
+      <child link="${prefix}gripper_contactsensor_link_1"/>
+    </joint>
+<!-- COLLISION/BUMPER SENSOR 2 LINK JOINT PLUGIN-->
+    <link name="${prefix}gripper_contactsensor_link_2">
+      <inertial >
+            <origin xyz="0 0 0" rpy="0 0 0"/>
+            <mass value="0.0001" />
+            <inertia ixx="1.6e-08" ixy="0.0" ixz="0.0" iyy="1.6e-08" iyz="0.0" izz="1.6e-08"/>
+        </inertial>
+        <collision>
+            <origin xyz="0 0 0" rpy="0 0 0"/>
+            <geometry>
+                <box size="0.02 0.02 0.0001"/>
+            </geometry>
+        </collision>
+        <visual>
+            <origin rpy="0.0 0 0" xyz="0 0 0"/>
+            <geometry>
+                <box size="0.02 0.02 0.0001"/>
+            </geometry>
+            <material name="red">
+              <color rgba="1.0 0 0 1.0"/>
+          </material>
+        </visual>
+    </link>
+    <joint name="${prefix}gripper_contactsensor_link_2_joint" type="fixed">
+      <origin xyz="0.019 0.296 0.0" rpy="1.570796325 0 0"/>
+      <parent link="${prefix}wrist_3_link"/>
+      <child link="${prefix}gripper_contactsensor_link_2"/>
+    </joint>
     <!-- INTEL REALSENSE DEPTH CAMERA -->
     <joint name="${prefix}camera_rgb_joint" type="fixed">

Commit message: add vacumm gripper

File: Pickbot_with_moveit/universal_robot/ur_description/urdf/ur.gazebo.xacro (robot description, xacro)
@@ -65,4 +65,23 @@
       </sensor>
     </gazebo>
+<!-- GRIPPER -->
+    <gazebo reference="${prefix}vacuum_gripper_link">
+      <material>Gazebo/Black</material>
+    </gazebo>
+    <gazebo>
+      <plugin name="ros_vacuum_gripper" filename="libROSVacuumGripperPlugin.so">
+        <grasp_check>
+          <detach_steps>40</detach_steps>
+          <attach_steps>1</attach_steps>
+          <min_contact_count>1</min_contact_count>
+        </grasp_check>
+        <!-- <xacro:insert_block name="drops_info" /> -->
+        <suction_cup_link>vacuum_gripper_link</suction_cup_link>
+        <!-- ROS -->
+        <robot_namespace>/pickbot</robot_namespace>
+        <control_topic>gripper/control</control_topic>
+        <state_topic>gripper/state</state_topic>
+      </plugin>
+    </gazebo>
     <!-- INTEL REALSENSE DEPTH CAMERA -->
     <gazebo reference="${prefix}camera_link2">

File: Pickbot_with_moveit/universal_robot/ur_description/urdf/ur10.urdf.xacro (robot description, xacro)
@@ -372,4 +372,39 @@
       <child link="${prefix}gripper_contactsensor_link_2"/>
     </joint>
+<!-- GRIPPER -->
+    <link name="${prefix}vacuum_gripper_link">
+      <inertial>
+        <origin xyz="0 0.0025 0" rpy="0 0 1.57"/>
+        <inertia ixx="0.0000063" ixy="0" ixz="0"
+                  iyy="0.0000063" iyz="0"
+                  izz="0.000025" />
+        <mass value="0.01" />
+      </inertial>
+      <visual>
+        <origin xyz="0 0.0025 0" rpy="0 0 1.57"/>
+        <geometry>
+          <box size="0.005 0.005 0.0001"/>
+          <!-- <cylinder radius="0.05" length="0.01"/> -->
+        </geometry>
+        <material name="SomeColor">
+          <color rgba="1.0 0.0 0.0 1.0"/>
+        </material>
+      </visual>
+      <collision>
+        <origin xyz="0 0.0025 0" rpy="0 0 1.57"/>
+        <geometry>
+          <box size="0.005 0.005 0.0001"/>
+          <!-- <cylinder radius="0.05" length="0.01"/> -->
+        </geometry>
+      </collision>
+    </link>
+    <joint name="${prefix}vacuum_gripper_joint" type="revolute">
+      <origin xyz="0 0.296 0" rpy="1.570797 0.0 0.0" />
+      <axis xyz="0 0 1" />
+      <limit lower="0" upper="0" effort="0" velocity="0" />
+      <parent link="${prefix}wrist_3_link" />
+      <child link="${prefix}vacuum_gripper_link" />
+      <dynamics damping="0.0" friction="0.0"/>
+    </joint>
     <!-- INTEL REALSENSE DEPTH CAMERA -->
     <joint name="${prefix}camera_rgb_joint" type="fixed">
