Commit message: add vacuum gripper to robot

File: Pickbot_with_moveit/universal_robot/ur_description/urdf/ur10.urdf.xacro (robot description, xacro)
@@ -70,4 +70,5 @@
       </visual>
       <collision>
+        <origin xyz="0 0 0" rpy="0 0 0"/>
         <geometry>
           <mesh filename="package://ur_description/meshes/ur10/collision/base.stl"/>
@@ -93,4 +94,5 @@
     <link name="${prefix}shoulder_link">
       <visual>
+        <origin xyz="0 0 0" rpy="0 0 0"/>
         <geometry>
           <mesh filename="package://ur_description/meshes/ur10/visual/shoulder.dae"/>
@@ -101,4 +103,5 @@
       </visual>
       <collision>
+        <origin xyz="0 0 0" rpy="0 0 0"/>
         <geometry>
           <mesh filename="package://ur_description/meshes/ur10/collision/shoulder.stl"/>
@@ -155,5 +158,6 @@
     <link name="${prefix}forearm_link">
       <visual>
-         <geometry>
+        <origin rpy="0.0 0.0 0.0" xyz="0.0 0.0 0.0"/>
+        <geometry>
           <mesh filename="package://ur_description/meshes/ur10/visual/forearm.dae"/>
         </geometry>
@@ -163,4 +167,5 @@
       </visual>
       <collision>
+        <origin rpy="0.0 0.0 0.0" xyz="0.0 0.0 0.0"/>
         <geometry>
           <mesh filename="package://ur_description/meshes/ur10/collision/forearm.stl"/>
@@ -186,4 +191,5 @@
     <link name="${prefix}wrist_1_link">
       <visual>
+        <origin rpy="0.0 0.0 0.0" xyz="0.0 0.0 0.0"/>
         <geometry>
           <mesh filename="package://ur_description/meshes/ur10/visual/wrist1.dae"/>
@@ -194,4 +200,5 @@
       </visual>
       <collision>
+        <origin rpy="0.0 0.0 0.0" xyz="0.0 0.0 0.0"/>
         <geometry>
           <mesh filename="package://ur_description/meshes/ur10/collision/wrist1.stl"/>
@@ -267,12 +274,24 @@
       <parent link="${prefix}wrist_3_link" />
       <child link = "${prefix}ee_link" />
-      <origin xyz="0.0 ${wrist_3_length} 0.0" rpy="0.0 0.0 ${pi/2.0}" />
+      <!-- <origin xyz="0.0 ${wrist_3_length} 0.0" rpy="0.0 0.0 ${pi/2.0}" /> -->
+      <origin xyz="-0.109 0.0652 -0.099" rpy="1.570796325 -1.570796325 0.0"/>
     </joint>
     <link name="${prefix}ee_link">
-      <collision>
-        <geometry>
-          <box size="0.01 0.01 0.01"/>
-        </geometry>
-        <origin rpy="0 0 0" xyz="-0.01 0 0"/>
+      <visual>
+        <origin rpy="0.0 0.0 0.0" xyz="0.0 0.0 0.0"/>
+        <geometry>
+          <mesh filename="package://pickbot_simulation/meshes/ur10/visual/Pickbot_Gripper.dae" scale="0.001 0.001 0.001"/>
+        </geometry>
+        <material name="LightGrey">
+          <color rgba="0.8 0.1 0.3 1.0"/>
+        </material>
+      </visual>
+      <collision>
+        <geometry>
+          <!-- <box size="0.01 0.01 0.01"/> -->
+          <mesh filename="package://ur_description/meshes/ur10/collision/Pickbot_Gripper.stl" scale="0.001 0.001 0.001"/>
+        </geometry>
+        <!-- <origin rpy="0 0 0" xyz="-0.01 0 0"/> -->
+        <origin rpy="0.0 0.0 0.0" xyz="0.0 0.0 0.0"/>
       </collision>
     </link>

Commit message: finetunining position of the onArm_camera

File: Pickbot_with_moveit/universal_robot/ur_description/urdf/ur10.urdf.xacro (robot description, xacro)
@@ -412,5 +412,5 @@
       <!-- <parent link="base_link"/> fixed camera -->
       <!-- <origin rpy="0 -1.57 -1.57" xyz="0 0.21 0.078"/> -->
-      <origin rpy="0 -0.9 1.57" xyz="0 0.21 -0.078"/>
+      <origin rpy="0 -0.4 1.57" xyz="0 0.21 -0.078"/>
       <parent link="${prefix}wrist_3_link"/>
       <child link="${prefix}camera_rgb_frame"/>
