Commit message: make the moveit aware of the environment

File: universal_robot/ur_description/urdf/ur.gazebo.xacro (robot description, xacro)
@@ -23,4 +23,12 @@
       <selfCollide>true</selfCollide>
     </gazebo>
+  <gazebo>
+    <plugin filename="libgazebo_ros_moveit_planning_scene.so" name="gazebo_ros_moveit_planning_scene">
+      <topicName>/planning_scene</topicName>
+      <sceneName>pickbot_planning</sceneName>
+      <robotName>ur10</robotName>
+      <updatePeriod>0.5</updatePeriod>
+    </plugin>
+  </gazebo>
     <!-- COLLISION/BUMPER SENSOR 1 LINK JOINT PLUGIN-->
     <gazebo reference="${prefix}gripper_contactsensor_link_1">

File: universal_robot/ur_description/urdf/ur10_joint_limited_robot.urdf.xacro (robot description, xacro)
@@ -21,5 +21,5 @@
     <parent link="world" />
     <child link = "base_link" />
-    <origin xyz="0.0 0.0 0.0" rpy="0.0 0.0 0.0" />
+    <origin xyz="0.0 0.0 1.01558" rpy="0.0 0.0 0.0" />
   </joint>
 </robot>

File: universal_robot/ur_description/urdf/ur10_robot.urdf.xacro (robot description, xacro)
@@ -15,5 +15,5 @@
     <parent link="world" />
     <child link = "base_link" />
-    <origin xyz="0.0 0.0 0.0" rpy="0.0 0.0 0.0" />
+    <origin xyz="0.0 0.0 1.01558" rpy="0.0 0.0 0.0" />
   </joint>
 </robot>

Commit message: moveit working with env-collision objects now

File: universal_robot/ur_description/urdf/ur.gazebo.xacro (robot description, xacro)
@@ -23,12 +23,12 @@
       <selfCollide>true</selfCollide>
     </gazebo>
-  <gazebo>
-    <plugin filename="libgazebo_ros_moveit_planning_scene.so" name="gazebo_ros_moveit_planning_scene">
-      <topicName>/planning_scene</topicName>
-      <sceneName>pickbot_planning</sceneName>
-      <robotName>ur10</robotName>
-      <updatePeriod>0.5</updatePeriod>
-    </plugin>
-  </gazebo>
+    <gazebo>
+      <plugin filename="libgazebo_ros_moveit_planning_scene.so" name="gazebo_ros_moveit_planning_scene">
+        <topicName>/planning_scene</topicName>
+        <sceneName>pickbot_planning</sceneName>
+        <robotName>ur10</robotName>
+        <updatePeriod>5000</updatePeriod>
+      </plugin>
+    </gazebo>
     <!-- COLLISION/BUMPER SENSOR 1 LINK JOINT PLUGIN-->
     <gazebo reference="${prefix}gripper_contactsensor_link_1">

File: universal_robot/ur_description/urdf/ur10_joint_limited_robot.urdf.xacro (robot description, xacro)
@@ -21,5 +21,5 @@
     <parent link="world" />
     <child link = "base_link" />
-    <origin xyz="0.0 0.0 1.01558" rpy="0.0 0.0 0.0" />
+    <origin xyz="0.0 0.0 1.12" rpy="0.0 0.0 0.0" />
   </joint>
 </robot>

File: universal_robot/ur_description/urdf/ur10_robot.urdf.xacro (robot description, xacro)
@@ -15,5 +15,5 @@
     <parent link="world" />
     <child link = "base_link" />
-    <origin xyz="0.0 0.0 1.01558" rpy="0.0 0.0 0.0" />
+    <origin xyz="0.0 0.0 1.12" rpy="0.0 0.0 0.0" />
   </joint>
 </robot>
