Commit message: add dummy_vaccum_gripper as end_effector for moveit

File: universal_robot/ur_description/urdf/ur.transmission.xacro (robot description, xacro)
@@ -56,4 +56,13 @@
       </actuator>
     </transmission>
+<!--    <transmission name="${prefix}vacuum_gripper_trans">-->
+<!--      <type>transmission_interface/SimpleTransmission</type>-->
+<!--      <joint name="${prefix}vacuum_gripper_joint">-->
+<!--        <hardwareInterface>${hw_interface}</hardwareInterface>-->
+<!--      </joint>-->
+<!--      <actuator name="${prefix}vacuum_gripper_motor">-->
+<!--        <mechanicalReduction>1</mechanicalReduction>-->
+<!--      </actuator>-->
+<!--    </transmission>-->
   </xacro:macro>
 </robot>

File: universal_robot/ur_description/urdf/ur10.urdf.xacro (robot description, xacro)
@@ -433,5 +433,5 @@
     </link>
     <joint name="${prefix}dummy_vacuum_gripper_joint" type="fixed">
-      <origin xyz="0 0.297 0.0" rpy="1.570797 0 0"/>
+      <origin xyz="0 0.2965 0.0" rpy="1.570797 0 0"/>
       <parent link="${prefix}wrist_3_link"/>
       <child link="${prefix}dummy_vacuum_gripper_link"/>
