Commit message: change vacuum_gripper_joint type from revolute to fixed

File: universal_robot/ur_description/urdf/ur10.urdf.xacro (robot description, xacro)
@@ -399,5 +399,5 @@
       </collision>
     </link>
-    <joint name="${prefix}vacuum_gripper_joint" type="revolute">
+    <joint name="${prefix}vacuum_gripper_joint" type="fixed">
       <origin xyz="0 0.296 0" rpy="1.570797 0.0 0.0" />
       <axis xyz="0 0 1" />

Commit message: change vacuum_gripper_joint back to revolute

File: universal_robot/ur_description/urdf/ur10.urdf.xacro (robot description, xacro)
@@ -399,5 +399,5 @@
       </collision>
     </link>
-    <joint name="${prefix}vacuum_gripper_joint" type="fixed">
+    <joint name="${prefix}vacuum_gripper_joint" type="revolute">
       <origin xyz="0 0.296 0" rpy="1.570797 0.0 0.0" />
       <axis xyz="0 0 1" />

Commit message: add <safety_controller> tag to constrain the joint_limit

File: universal_robot/ur_description/urdf/ur10.urdf.xacro (robot description, xacro)
@@ -91,4 +91,5 @@
       </xacro:if>
       <dynamics damping="0.0" friction="0.0"/>
+      <safety_controller k_velocity="10" k_position="10" soft_lower_limit="-2.0" soft_upper_limit="2.0" />
     </joint>
     <link name="${prefix}shoulder_link">
@@ -124,4 +125,5 @@
       </xacro:if>
       <dynamics damping="0.0" friction="0.0"/>
+      <safety_controller k_velocity="10" k_position="10" soft_lower_limit="-2.0" soft_upper_limit="2.0" />
     </joint>
     <link name="${prefix}upper_arm_link">
@@ -155,4 +157,5 @@
       </xacro:if>
       <dynamics damping="0.0" friction="0.0"/>
+      <safety_controller k_velocity="10" k_position="10" soft_lower_limit="-2.0" soft_upper_limit="2.0" />
     </joint>
     <link name="${prefix}forearm_link">
@@ -188,4 +191,5 @@
       </xacro:if>
       <dynamics damping="0.0" friction="0.0"/>
+      <safety_controller k_velocity="10" k_position="10" soft_lower_limit="-2.0" soft_upper_limit="2.0" />
     </joint>
     <link name="${prefix}wrist_1_link">
@@ -221,4 +225,5 @@
       </xacro:if>
       <dynamics damping="0.0" friction="0.0"/>
+      <safety_controller k_velocity="10" k_position="10" soft_lower_limit="-2.0" soft_upper_limit="2.0" />
     </joint>
     <link name="${prefix}wrist_2_link">
@@ -252,4 +257,5 @@
       </xacro:if>
       <dynamics damping="0.0" friction="0.0"/>
+      <safety_controller k_velocity="10" k_position="10" soft_lower_limit="-2.0" soft_upper_limit="2.0" />
     </joint>
     <link name="${prefix}wrist_3_link">
@@ -402,8 +408,9 @@
       <origin xyz="0 0.296 0" rpy="1.570797 0.0 0.0" />
       <axis xyz="0 0 1" />
-      <limit lower="0" upper="0" effort="0" velocity="0" />
+      <limit lower="0.0" upper="0.0" effort="0" velocity="0" />
       <parent link="${prefix}wrist_3_link" />
       <child link="${prefix}vacuum_gripper_link" />
       <dynamics damping="0.0" friction="0.0"/>
+      <safety_controller k_velocity="10" k_position="10" soft_lower_limit="0.0" soft_upper_limit="0.0" />
     </joint>
     <!-- INTEL REALSENSE DEPTH CAMERA -->

Commit message: add dummy_vacuum_gripper to robot

File: universal_robot/ur_description/urdf/ur10.urdf.xacro (robot description, xacro)
@@ -414,4 +414,27 @@
 <!--      <safety_controller k_velocity="10" k_position="10" soft_lower_limit="0.0" soft_upper_limit="0.0" />-->
     </joint>
+    <link name="${prefix}dummy_vacuum_gripper_link">
+        <inertial>
+          <origin xyz="0 0.0025 0" rpy="0 0 1.57"/>
+          <inertia ixx="0.0000063" ixy="0" ixz="0"
+                  iyy="0.0000063" iyz="0"
+                  izz="0.000025" />
+          <mass value="0.01" />
+        </inertial>
+        <visual>
+          <origin xyz="0 0.0025 0" rpy="0 0 1.57"/>
+          <geometry>
+            <box size="0.003 0.003 0.0001"/>
+          </geometry>
+          <material name="SomeColor">
+            <color rgba="1.0 0.0 0.0 1.0"/>
+          </material>
+      </visual>
+    </link>
+    <joint name="${prefix}dummy_vacuum_gripper_joint" type="fixed">
+      <origin xyz="0 0.297 0.0" rpy="1.570797 0 0"/>
+      <parent link="${prefix}wrist_3_link"/>
+      <child link="${prefix}dummy_vacuum_gripper_link"/>
+    </joint>
     <!-- INTEL REALSENSE DEPTH CAMERA -->
     <joint name="${prefix}camera_rgb_joint" type="fixed">

Commit message: finetune the position of dummy_vacuum_gripper

File: universal_robot/ur_description/urdf/ur10.urdf.xacro (robot description, xacro)
@@ -433,5 +433,5 @@
     </link>
     <joint name="${prefix}dummy_vacuum_gripper_joint" type="fixed">
-      <origin xyz="0 0.2965 0.0" rpy="1.570797 0 0"/>
+      <origin xyz="0 0.29615 0.0" rpy="1.570797 0 0"/>
       <parent link="${prefix}wrist_3_link"/>
       <child link="${prefix}dummy_vacuum_gripper_link"/>
